Commit message: fix ur urdf for jazzy

File: uclv_urdf_demo/urdf/ur.urdf.xacro (robot description, xacro)
@@ -1,9 +1,11 @@
 <?xml version="1.0"?>
-<robot xmlns:xacro="http://wiki.ros.org/xacro" name="ur_robot">
+<robot xmlns:xacro="http://wiki.ros.org/xacro" name="ur_robot"> <!-- <- we are not using $(arg name) -->
+   <!-- robot name parameter -->
+   <xacro:arg name="name" default="ur"/>
    <!-- import main macro -->
    <xacro:include filename="$(find ur_description)/urdf/ur_macro.xacro"/>
-   <!-- possible 'ur_type' values: ur3, ur3e, ur5, ur5e, ur10, ur10e, ur16e, ur20, ur30 -->
+   <!-- possible 'ur_type' values: ur3, ur3e, ur5, ur5e, ur7e, ur10, ur10e, ur12e, ur16e, ur20, ur30 -->
    <!-- the default value should raise an error in case this was called without defining the type -->
-   <xacro:arg name="ur_type" default="ur5e"/>
+   <xacro:arg name="ur_type" default="ur5e"/> <!-- <- Modified! -->
    <!-- parameters -->
    <xacro:arg name="tf_prefix" default="" />
@@ -12,13 +14,9 @@
    <xacro:arg name="physical_params" default="$(find ur_description)/config/$(arg ur_type)/physical_parameters.yaml"/>
    <xacro:arg name="visual_params" default="$(find ur_description)/config/$(arg ur_type)/visual_parameters.yaml"/>
-   <xacro:arg name="transmission_hw_interface" default=""/>
-   <xacro:arg name="safety_limits" default="false"/>
-   <xacro:arg name="safety_pos_margin" default="0.15"/>
-   <xacro:arg name="safety_k_position" default="20"/>
    <!-- create link fixed to the "world" -->
    <link name="world" />
    <!-- arm -->
    <xacro:ur_robot
-     name="ur_robot"
+     name="$(arg name)"
      tf_prefix="$(arg tf_prefix)"
      parent="world"
@@ -27,8 +25,4 @@
      physical_parameters_file="$(arg physical_params)"
      visual_parameters_file="$(arg visual_params)"
-     transmission_hw_interface="$(arg transmission_hw_interface)"
-     safety_limits="$(arg safety_limits)"
-     safety_pos_margin="$(arg safety_pos_margin)"
-     safety_k_position="$(arg safety_k_position)"
      >
      <origin xyz="0 0 0" rpy="0 0 0" />          <!-- position robot in the world -->

File: uclv_urdf_demo/urdf/ur_with_robotiq.urdf.xacro (robot description, xacro)
@@ -1,11 +1,13 @@
 <?xml version="1.0"?>
-<robot xmlns:xacro="http://wiki.ros.org/xacro" name="ur_robot">
-   <!-- import UR5 macro -->
+<robot xmlns:xacro="http://wiki.ros.org/xacro" name="ur_robot"> <!-- <- we are not using $(arg name) -->
+   <!-- robot name parameter -->
+   <xacro:arg name="name" default="ur"/>
+   <!-- import main macro -->
    <xacro:include filename="$(find ur_description)/urdf/ur_macro.xacro"/>
    <!-- import ROBOTIQ GRIPPER macro -->
    <xacro:include filename="$(find uclv_urdf_robotiq_demo)/urdf/robotiq_arg2f_140_macro.xacro" />
-   <!-- possible 'ur_type' values: ur3, ur3e, ur5, ur5e, ur10, ur10e, ur16e, ur20, ur30 -->
+   <!-- possible 'ur_type' values: ur3, ur3e, ur5, ur5e, ur7e, ur10, ur10e, ur12e, ur16e, ur20, ur30 -->
    <!-- the default value should raise an error in case this was called without defining the type -->
-   <xacro:arg name="ur_type" default="ur5e"/>
+   <xacro:arg name="ur_type" default="ur5e"/> <!-- <- Modified! -->
    <!-- parameters -->
    <xacro:arg name="tf_prefix" default="" />
@@ -14,13 +16,9 @@
    <xacro:arg name="physical_params" default="$(find ur_description)/config/$(arg ur_type)/physical_parameters.yaml"/>
    <xacro:arg name="visual_params" default="$(find ur_description)/config/$(arg ur_type)/visual_parameters.yaml"/>
-   <xacro:arg name="transmission_hw_interface" default=""/>
-   <xacro:arg name="safety_limits" default="false"/>
-   <xacro:arg name="safety_pos_margin" default="0.15"/>
-   <xacro:arg name="safety_k_position" default="20"/>
    <!-- create link fixed to the "world" -->
    <link name="world" />
    <!-- arm -->
    <xacro:ur_robot
-     name="ur_robot"
+     name="$(arg name)"
      tf_prefix="$(arg tf_prefix)"
      parent="world"
@@ -29,8 +27,4 @@
      physical_parameters_file="$(arg physical_params)"
      visual_parameters_file="$(arg visual_params)"
-     transmission_hw_interface="$(arg transmission_hw_interface)"
-     safety_limits="$(arg safety_limits)"
-     safety_pos_margin="$(arg safety_pos_margin)"
-     safety_k_position="$(arg safety_k_position)"
      >
      <origin xyz="0 0 0" rpy="0 0 0" />          <!-- position robot in the world -->
@@ -38,12 +32,12 @@
    <joint name="$(arg tf_prefix)flange_gripper_joint" type="fixed">
         <!-- Sometimes you need to modify the origin of the fixed joints -->
-        <origin xyz="0 0 0" rpy="0 0 0" />
-        <!-- <origin xyz="0 0 0" rpy="0 ${pi/2} 0" /> -->
+        <!-- <origin xyz="0 0 0" rpy="0 0 0" /> -->
+        <origin xyz="0 0 0" rpy="0 ${pi/2} 0" />
         <parent link="$(arg tf_prefix)flange" />
         <child link="$(arg tf_prefix)robotiq_base_link" />
-    </joint>
+   </joint>
    <!-- gripper -->
-  <xacro:robotiq_arg2f_140
-    prefix="$(arg tf_prefix)robotiq_"
-  />
+   <xacro:robotiq_arg2f_140
+     prefix="$(arg tf_prefix)robotiq_"
+   />
 </robot>
