Commit message: add tf_prefix

File: uclv_urdf_demo/urdf/ur_with_robotiq.urdf.xacro (robot description, xacro)
@@ -40,5 +40,5 @@
         <origin xyz="0 0 0" rpy="0 0 0" />
         <!-- <origin xyz="0 0 0" rpy="0 ${pi/2} 0" /> -->
-        <parent link="flange" />
+        <parent link="$(arg tf_prefix)flange" />
         <child link="$(arg tf_prefix)robotiq_base_link" />
     </joint>

Commit message: in this version you have to manually modify the origin of the tool

File: uclv_urdf_demo/urdf/ur_with_robotiq.urdf.xacro (robot description, xacro)
@@ -32,6 +32,6 @@
    <joint name="$(arg tf_prefix)flange_gripper_joint" type="fixed">
         <!-- Sometimes you need to modify the origin of the fixed joints -->
-        <!-- <origin xyz="0 0 0" rpy="0 0 0" /> -->
-        <origin xyz="0 0 0" rpy="0 ${pi/2} 0" />
+        <origin xyz="0 0 0" rpy="0 0 0" />
+        <!-- <origin xyz="0 0 0" rpy="0 ${pi/2} 0" /> -->
         <parent link="$(arg tf_prefix)flange" />
         <child link="$(arg tf_prefix)robotiq_base_link" />
